Commit message: cambios en los launch e implementacion de tutorialbase de urdf

File: src/urdf_sdf/urdf/test.urdf (robot description, URDF)
Before this commit: robot tubo, 2 links, 1 joints
Links:
- link base_link: mass 10 -> None; geometry visual cylinder length=0.6 radius=0.2
Joints:
- joint base_to_right_leg: axis 0.0 1.0 0.0 -> (none); origin xyz=0 -0.22 0.25 -> (none); type continuous -> fixed
